Commit message: update_robot_model

File: urdf/aynasiz_robot.xacro (robot description, xacro)
@@ -7,9 +7,9 @@
   <xacro:include filename="$(find aynasiz_description)/urdf/diferansiyel.xacro"/>
   <xacro:sase />
-  <xacro:ust_sase xyz_konum="0 0 0.04" rpy_konum="0 0 0" />
-  <xacro:tekerler xyz_konum="0 0.06 0.0055" rpy_konum="0 0 0" yon="left"/>
-  <xacro:tekerler xyz_konum="0 -0.06 0.0055" rpy_konum="0 0 0" yon="right"/>
-  <xacro:sarhos_tekerler xyz_konum="0.09 0 -0.0110" rpy_konum="0 0 0" yon="forward_chaster_wheel"/>
-  <xacro:sarhos_tekerler xyz_konum="-0.09 0 -0.0110" rpy_konum="0 0 0" yon="backward_chaster_wheel"/>
+  <xacro:ust_sase xyz_konum="0 0 0.05" rpy_konum="0 0 0" />
+  <xacro:tekerler xyz_konum="0 0.06 0.01" rpy_konum="0 0 0" yon="left"/>
+  <xacro:tekerler xyz_konum="0 -0.06 0.01" rpy_konum="0 0 0" yon="right"/>
+  <xacro:sarhos_tekerler xyz_konum="0.09 0 -0.00925" rpy_konum="0 0 0" yon="forward_chaster_wheel"/>
+  <xacro:sarhos_tekerler xyz_konum="-0.09 0 -0.00925" rpy_konum="0 0 0" yon="backward_chaster_wheel"/>
   <xacro:diferansiyel />
 </robot>

File: urdf/diferansiyel.xacro (robot description, xacro)
@@ -7,7 +7,7 @@
 	    <updateRate>10.0</updateRate>
 	    <!-- Name of left joint, defaults to `left_joint` -->
-	    <leftJoint>wheel_left_base</leftJoint>
+	    <leftJoint>wheel_left_joint</leftJoint>
 	    <!-- Name of right joint, defaults to `right_joint` -->
-	    <rightJoint>wheel_right_base</rightJoint>
+	    <rightJoint>wheel_right_joint</rightJoint>
 	    <!-- The distance from the center of one wheel to the other, in meters, defaults to 0.34 m -->
 	    <wheelSeparation>0.12</wheelSeparation>
@@ -17,5 +17,5 @@
 	    <wheelAcceleration>0.0</wheelAcceleration>
 	    <!-- Maximum torque which the wheels can produce, in Nm, defaults to 5 Nm -->
-	    <wheelTorque>16.35</wheelTorque>
+	    <wheelTorque>5</wheelTorque>
 	    <!-- Topic to receive geometry_msgs/Twist message commands, defaults to `cmd_vel` -->
 	    <commandTopic>cmd_vel</commandTopic>
@@ -27,5 +27,5 @@
 	    <robotBaseFrame>base_link</robotBaseFrame>
 	    <!-- Odometry source, 0 for ENCODER, 1 for WORLD, defaults to WORLD -->
-	    <odometrySource>0</odometrySource>
+	    <odometrySource>1</odometrySource>
 	    <!-- Set to true to publish transforms for the wheel links, defaults to false -->
 	    <publishWheelTF>true</publishWheelTF>

File: urdf/tekerlekler.xacro (robot description, xacro)
@@ -17,5 +17,5 @@
     <xacro:cylinder_inertial radius="0.03" length="0.0011" mass="0.04"/>
   </link>
-  <joint name="wheel_${yon}_base" type="continuous">
+  <joint name="wheel_${yon}_joint" type="continuous">
     <origin xyz="${xyz_konum}" rpy="${rpy_konum}"/>
     <parent link="base_link"/>
@@ -43,5 +43,5 @@
     <xacro:sphere_inertial radius="0.0105" mass="0.04"/>
   </link>
-  <joint name="caster_wheel_${yon}_base" type="continuous">
+  <joint name="caster_wheel_${yon}_joint" type="continuous">
     <origin xyz="${xyz_konum}" rpy="${rpy_konum}"/>
     <parent link="base_link"/>
@@ -50,5 +50,5 @@
   </joint>
   <gazebo reference="caster_wheel_${yon}_link">
-    <material value="Gazebo/White"/>
+    <material value="Gazebo/black"/>
   </gazebo>
   </xacro:macro>

File: urdf/ust_sase.xacro (robot description, xacro)
@@ -15,4 +15,6 @@
         </geometry>
       </visual>
+    <xacro:cylinder_inertial radius="0.02" length="0.01" mass="0.2"/>
+    </link>
     <joint name="ust_sase_joint" type="fixed">
         <origin xyz="${xyz_konum}" rpy="${rpy_konum}"/>
@@ -21,6 +23,4 @@
         <axis xyz="0 0 0"/>
     </joint>
-    <xacro:cylinder_inertial radius="0.02" length="0.01" mass="0.2"/>
-    </link>
     <gazebo reference="base_link">
       <material value="Gazebo/Blue"/>
